Commit message: Working Descriptions for Gazebo

File: franka_description/robots/panda_arm.urdf.xacro (robot description, xacro)
@@ -6,4 +6,5 @@
   <xacro:arg name="use_fake_hardware" default="false"/>
   <xacro:arg name="fake_sensor_commands" default="false"/>
+  <link name="world" />
   <xacro:include filename="$(find franka_description)/robots/panda_arm.xacro"/>
   <xacro:panda_arm arm_id="$(arg arm_id)" safety_distance="0.03"/>
@@ -12,5 +13,8 @@
     <xacro:hand ns="$(arg arm_id)" rpy="0 0 ${-pi/4}" connected_to="$(arg arm_id)_link8" safety_distance="0.03"/>
   </xacro:if>
+  <xacro:include filename="$(find franka_description)/robots/manipulator.gazebo.xacro" />
+  <xacro:include filename="$(find franka_description)/robots/manipulator.control.xacro" />
   <xacro:include filename="$(find franka_description)/robots/panda_arm.ros2_control.xacro"/>
-  <xacro:panda_arm_ros2_control ns="$(arg arm_id)" robot_ip="$(arg robot_ip)" use_fake_hardware="$(arg use_fake_hardware)" fake_sensor_commands="$(arg fake_sensor_commands)"/>
+  <!--<xacro:panda_arm_ros2_control ns="$(arg arm_id)" robot_ip="$(arg robot_ip)" use_fake_hardware="$(arg use_fake_hardware)" fake_sensor_commands="$(arg fake_sensor_commands)"/>
+  -->
 </robot>

File: franka_description/robots/panda_arm.xacro (robot description, xacro)
@@ -1,4 +1,58 @@
 <?xml version='1.0' encoding='utf-8'?>
 <robot xmlns:xacro="http://www.ros.org/wiki/xacro" name="panda">
+<!-- ADDED -->
+<!--
+  <link name="dummy_link">
+    <visual>
+      <geometry>
+        <box size="0.01 0.01 0.01"/>
+      </geometry>
+    </visual>
+  </link>
+  <joint name="dummy_joint" type="fixed">
+    <parent link="dummy_link"/>
+    <child link="panda_link0"/>
+  </joint>
+  -->
+  <!--Correct
+  masses-->
+  <xacro:property name="mass_link0" value="3.06357" />
+  <xacro:property name="mass_link1" value="2.34471" />
+  <xacro:property name="mass_link2" value="2.36414" />
+  <xacro:property name="mass_link3" value="2.38050" />
+  <xacro:property name="mass_link4" value="2.42754" />
+  <xacro:property name="mass_link5" value="3.49611" />
+  <xacro:property name="mass_link6" value="1.46736" />
+  <xacro:property name="mass_link7" value="0.45606" />
+  <xacro:property name="mass_link8" value="0.001" />
+  <!-- Wrong masses to test adaptability of the algorithms, on purpose off by 20% -->
+  <!--xacro:property
+  name="mass_link0" value="3.66357" />
+  <xacro:property name="mass_link1" value="2.04471" />
+  <xacro:property name="mass_link2" value="2.56414" />
+  <xacro:property name="mass_link3" value="2.48050" />
+  <xacro:property name="mass_link4" value="2.02754" />
+  <xacro:property name="mass_link5" value="3.09611" />
+  <xacro:property name="mass_link6" value="1.66736" />
+  <xacro:property name="mass_link7" value="0.75606" />
+  <xacro:property name="mass_link8" value="0.1" /-->
+  <xacro:property name="link0_cog" value="-0.029190 -0.000879 0.056603" />
+  <xacro:property name="link1_cog" value="0.000011 -0.031266 -0.069373" />
+  <xacro:property name="link2_cog" value="-0.000013 -0.070322 0.031178" />
+  <xacro:property name="link3_cog" value="0.044348 0.024928 -0.038130" />
+  <xacro:property name="link4_cog" value="-0.038550 0.039526 0.024716" />
+  <xacro:property name="link5_cog" value="-0.000064 0.038412 -0.109970" />
+  <xacro:property name="link6_cog" value="0.051002 0.006933 0.006169" />
+  <xacro:property name="link7_cog" value="0.010361 0.010360 0.079108" />
+ <xacro:macro name="cylinder_inertial" params="radius length mass *origin">
+    <inertial>
+      <mass value="${mass}" />
+      <xacro:insert_block name="origin" />
+      <inertia ixx="${0.0833333 * mass * (3 * radius * radius + length * length)}" ixy="0.0"
+        ixz="0.0"
+        iyy="${0.0833333 * mass * (3 * radius * radius + length * length)}" iyz="0.0"
+        izz="${0.5 * mass * radius * radius}" />
+    </inertial>
+  </xacro:macro>
   <!-- safety_distance: Minimum safety distance in [m] by which the collision volumes are expanded and which is enforced during robot motions -->
   <!-- arm_id: Namespace of the panda arm. Serves to differentiate between arms in case of multiple instances. -->
@@ -11,8 +65,17 @@
       </joint>
     </xacro:unless>
+    <xacro:property
+      name="joint_damping" value="1.0" />
+    <joint name="robot_to_world" type="fixed">
+      <parent link="world" />
+      <child link="${arm_id}_link0" />
+      <origin xyz="0.0 0.0 0.0" rpy="0.0 0.0 0.0" />
+      <dynamics damping="${joint_damping}" />
+    </joint>
+     <!--UNTIL HERE -->
     <link name="${arm_id}_link0">
       <visual>
         <geometry>
-          <mesh filename="package://${description_pkg}/meshes/visual/link0.dae"/>
+          <mesh filename="file://$(find franka_description)/meshes/visual/link0.dae"/>
         </geometry>
       </visual>
@@ -35,9 +98,14 @@
         </geometry>
       </collision>
+      <inertial>
+        <origin xyz="${link0_cog}" rpy="0 0 0" />
+        <mass value="${mass_link0}" />
+        <inertia ixx="0.009" iyy="0.0122" izz="0.0122" ixy="0.0" ixz="-0.00010" iyz="0.0" />
+      </inertial>
     </link>
     <link name="${arm_id}_link1">
       <visual>
         <geometry>
-          <mesh filename="package://${description_pkg}/meshes/visual/link1.dae"/>
+          <mesh filename="file://$(find franka_description)/meshes/visual/link1.dae"/>
         </geometry>
       </visual>
@@ -60,4 +128,9 @@
         </geometry>
       </collision>
+      <inertial>
+        <origin xyz="${link1_cog}" rpy="0 0 0" />
+        <mass value="${mass_link1}" />
+        <inertia ixx="0.01418" iyy="0.01181" izz="0.005515" ixy="0.0" ixz="0.0" iyz="0.00236" />
+      </inertial>
     </link>
     <joint name="${arm_id}_joint1" type="revolute">
@@ -72,5 +145,5 @@
       <visual>
         <geometry>
-          <mesh filename="package://${description_pkg}/meshes/visual/link2.dae"/>
+          <mesh filename="file://$(find franka_description)/meshes/visual/link2.dae"/>
         </geometry>
       </visual>
@@ -93,4 +166,9 @@
         </geometry>
       </collision>
+      <inertial>
+        <origin xyz="${link2_cog}" rpy="0 0 0" />
+        <mass value="${mass_link2}" />
+        <inertia ixx="0.014" ixy="0.0" ixz="0.0" iyy="0.0055" iyz="-0.0023" izz="0.01259" />
+      </inertial>
     </link>
     <joint name="${arm_id}_joint2" type="revolute">
@@ -105,5 +183,5 @@
       <visual>
         <geometry>
-          <mesh filename="package://${description_pkg}/meshes/visual/link3.dae"/>
+          <mesh filename="file://$(find franka_description)/meshes/visual/link3.dae"/>
         </geometry>
       </visual>
@@ -126,4 +204,10 @@
         </geometry>
       </collision>
+      <inertial>
+        <origin xyz="${link3_cog}" rpy="0 0 0" />
+        <mass value="${mass_link3}" />
+        <inertia ixx="0.00716" ixy="-0.00102" ixz="-0.02040" iyy="0.00920" iyz="-0.00102"
+          izz="0.007159" />
+      </inertial>
     </link>
     <joint name="${arm_id}_joint3" type="revolute">
@@ -138,5 +222,5 @@
       <visual>
         <geometry>
-          <mesh filename="package://${description_pkg}/meshes/visual/link4.dae"/>
+          <mesh filename="file://$(find franka_description)/meshes/visual/link4.dae"/>
         </geometry>
       </visual>
@@ -159,4 +243,10 @@
         </geometry>
       </collision>
+      <inertial>
+        <origin xyz="${link4_cog}" rpy="0 0 0" />
+        <mass value="${mass_link4}" />
+        <inertia ixx="0.008164" ixy="0.003061" ixz="0.00102" iyy="0.008165" iyz="0.00102"
+          izz="0.009185" />
+      </inertial>
     </link>
     <joint name="${arm_id}_joint4" type="revolute">
@@ -171,5 +261,5 @@
       <visual>
         <geometry>
-          <mesh filename="package://${description_pkg}/meshes/visual/link5.dae"/>
+          <mesh filename="file://$(find franka_description)/meshes/visual/link5.dae"/>
         </geometry>
       </visual>
@@ -210,4 +300,9 @@
         </geometry>
       </collision>
+      <inertial>
+        <origin xyz="${link5_cog}" rpy="0 0 0" />
+        <mass value="${mass_link5}" />
+        <inertia ixx="0.0307" ixy="0.0" ixz="0.0" iyy="0.02761" iyz="-0.0613" izz="0.00818" />
+      </inertial>
     </link>
     <joint name="${arm_id}_joint5" type="revolute">
@@ -222,5 +317,5 @@
       <visual>
         <geometry>
-          <mesh filename="package://${description_pkg}/meshes/visual/link6.dae"/>
+          <mesh filename="file://$(find franka_description)/meshes/visual/link6.dae"/>
         </geometry>
       </visual>
@@ -243,4 +338,9 @@
         </geometry>
       </collision>
+      <inertial>
+        <origin xyz="${link6_cog}" rpy="0 0 0" />
+        <mass value="${mass_link6}" />
+        <inertia ixx="0.00205" ixy="0.0" ixz="0.0" iyy="0.004089" iyz="0" izz="0.00490" />
+      </inertial>
     </link>
     <joint name="${arm_id}_joint6" type="revolute">
@@ -255,5 +355,5 @@
       <visual>
         <geometry>
-          <mesh filename="package://${description_pkg}/meshes/visual/link7.dae"/>
+          <mesh filename="file://$(find franka_description)/meshes/visual/link7.dae"/>
         </geometry>
       </visual>
@@ -276,4 +376,9 @@
         </geometry>
       </collision>
+      <inertial>
+        <origin xyz="0 0 0" rpy="0 0 0" />
+        <mass value="${mass_link7}" />
+        <inertia ixx="0.3" ixy="0.0" ixz="0.0" iyy="0.3" iyz="0.0" izz="0.3" />
+      </inertial>
     </link>
     <joint name="${arm_id}_joint7" type="revolute">
@@ -304,4 +409,9 @@
         </geometry>
       </collision>
+      <inertial>
+        <origin xyz="0 0 0" rpy="0 0 0" />
+        <mass value="${mass_link8}" />
+        <inertia ixx="0.3" ixy="0.0" ixz="0.0" iyy="0.3" iyz="0.0" izz="0.3" />
+      </inertial>
     </link>
     <joint name="${arm_id}_joint8" type="fixed">

Commit message: Removing unecessary files.

File: franka_description/robots/panda_arm.urdf.xacro (robot description, xacro)
@@ -6,5 +6,5 @@
   <xacro:arg name="use_fake_hardware" default="false"/>
   <xacro:arg name="fake_sensor_commands" default="false"/>
-  <link name="world" />
+  <link name="world"/>
   <xacro:include filename="$(find franka_description)/robots/panda_arm.xacro"/>
   <xacro:panda_arm arm_id="$(arg arm_id)" safety_distance="0.03"/>
@@ -16,5 +16,4 @@
   <xacro:include filename="$(find franka_description)/robots/manipulator.control.xacro" />
   <xacro:include filename="$(find franka_description)/robots/panda_arm.ros2_control.xacro"/>
-  <!--<xacro:panda_arm_ros2_control ns="$(arg arm_id)" robot_ip="$(arg robot_ip)" use_fake_hardware="$(arg use_fake_hardware)" fake_sensor_commands="$(arg fake_sensor_commands)"/>
-  -->
+  <xacro:panda_arm_ros2_control ns="$(arg arm_id)" robot_ip="$(arg robot_ip)" use_fake_hardware="$(arg use_fake_hardware)" fake_sensor_commands="$(arg fake_sensor_commands)"/>
 </robot>
