Commit message: Changing each joint to macro

File: franka_description/robots/manipulator.control.xacro (robot description, xacro)
@@ -10,4 +10,31 @@
             <plugin>gazebo_ros2_control/GazeboSystem</plugin>
         </hardware>
+        <xacro:macro name="joint_configuration" params="joint_name">
+            <joint name="${joint_name}">
+                <command_interface name="effort">
+                </command_interface>
+                <command_interface name="position">
+                </command_interface>
+                <state_interface name="position" />
+                <state_interface name="velocity" />
+                <state_interface name="effort" />
+            </joint>
+        </xacro:macro>
+        <xacro:property name="arm_id" value="panda" />
+        <xacro:joint_configuration joint_name="${arm_id}_joint1"/>
+        <xacro:joint_configuration joint_name="${arm_id}_joint2"/>
+        <xacro:joint_configuration joint_name="${arm_id}_joint3"/>
+        <xacro:joint_configuration joint_name="${arm_id}_joint4"/>
+        <xacro:joint_configuration joint_name="${arm_id}_joint5"/>
+        <xacro:joint_configuration joint_name="${arm_id}_joint6"/>
+        <xacro:joint_configuration joint_name="${arm_id}_joint7"/>
+        <!--
+        <xacro:configure_joint joint_name="${ns}_joint1" initial_position="0.0}"/>
+        <xacro:configure_joint joint_name="${ns}_joint2" initial_position="${-pi/4}"/>
+        <xacro:configure_joint joint_name="${ns}_joint3" initial_position="0.0"/>
+        <xacro:configure_joint joint_name="${ns}_joint4" initial_position="${-3*pi/4}"/>
+        <xacro:configure_joint joint_name="${ns}_joint5" initial_position="0.0"/>
+        <xacro:configure_joint joint_name="${ns}_joint6" initial_position="${pi/2}"/>
+        <xacro:configure_joint joint_name="${ns}_joint7" initial_position="${pi/4}"/>
         <joint name="panda_joint1">
             <command_interface name="effort">
@@ -73,4 +100,5 @@
             <state_interface name="effort" />
         </joint>
+        -->
     </ros2_control>
 </robot>

Commit message: Bug Fix to change the initial position

File: franka_description/robots/manipulator.control.xacro (robot description, xacro)
@@ -10,11 +10,11 @@
             <plugin>gazebo_ros2_control/GazeboSystem</plugin>
         </hardware>
-        <xacro:macro name="joint_configuration" params="joint_name">
+        <xacro:macro name="joint_configuration" params="joint_name initial_position">
             <joint name="${joint_name}">
-                <command_interface name="effort">
-                </command_interface>
-                <command_interface name="position">
-                </command_interface>
-                <state_interface name="position" />
+                <command_interface name="effort" />
+                <command_interface name="position"/>
+                <state_interface name="position">
+                    <param name="initial_value">${initial_position}</param>
+                </state_interface>
                 <state_interface name="velocity" />
                 <state_interface name="effort" />
@@ -22,11 +22,11 @@
         </xacro:macro>
         <xacro:property name="arm_id" value="panda" />
-        <xacro:joint_configuration joint_name="${arm_id}_joint1"/>
-        <xacro:joint_configuration joint_name="${arm_id}_joint2"/>
-        <xacro:joint_configuration joint_name="${arm_id}_joint3"/>
-        <xacro:joint_configuration joint_name="${arm_id}_joint4"/>
-        <xacro:joint_configuration joint_name="${arm_id}_joint5"/>
-        <xacro:joint_configuration joint_name="${arm_id}_joint6"/>
-        <xacro:joint_configuration joint_name="${arm_id}_joint7"/>
+        <xacro:joint_configuration joint_name="${arm_id}_joint1" initial_position="0.0"/>
+        <xacro:joint_configuration joint_name="${arm_id}_joint2" initial_position="${+pi/4}"/>
+        <xacro:joint_configuration joint_name="${arm_id}_joint3" initial_position="0.0"/>
+        <xacro:joint_configuration joint_name="${arm_id}_joint4" initial_position="${-3*pi/4}"/>
+        <xacro:joint_configuration joint_name="${arm_id}_joint5" initial_position="0.0"/>
+        <xacro:joint_configuration joint_name="${arm_id}_joint6" initial_position="${pi/2}"/>
+        <xacro:joint_configuration joint_name="${arm_id}_joint7" initial_position="${pi/4}"/>
         <!--
         <xacro:configure_joint joint_name="${ns}_joint1" initial_position="0.0}"/>
@@ -51,5 +51,7 @@
             <command_interface name="position">
             </command_interface>
-            <state_interface name="position" />
+            <state_interface name="position">
+                    <param name="initial_position">${initial_position}</param>
+            </state_interface>
             <state_interface name="velocity" />
             <state_interface name="effort" />

Commit message: Using initial_position.yaml for starting joint angels of robot

File: franka_description/robots/manipulator.control.xacro (robot description, xacro)
@@ -22,19 +22,15 @@
         </xacro:macro>
         <xacro:property name="arm_id" value="panda" />
-        <xacro:joint_configuration joint_name="${arm_id}_joint1" initial_position="0.0"/>
-        <xacro:joint_configuration joint_name="${arm_id}_joint2" initial_position="${+pi/4}"/>
-        <xacro:joint_configuration joint_name="${arm_id}_joint3" initial_position="0.0"/>
-        <xacro:joint_configuration joint_name="${arm_id}_joint4" initial_position="${-3*pi/4}"/>
-        <xacro:joint_configuration joint_name="${arm_id}_joint5" initial_position="0.0"/>
-        <xacro:joint_configuration joint_name="${arm_id}_joint6" initial_position="${pi/2}"/>
-        <xacro:joint_configuration joint_name="${arm_id}_joint7" initial_position="${pi/4}"/>
+        <xacro:arg name="initial_joint_values_path" default=""/> <!-- Need argument to get from launch file -->
+        <xacro:property name="jv_path" value="$(arg initial_joint_values_path)"/> <!-- Need seperate property for xacro inorder processing -->
+        <xacro:property name="jv" value="${xacro.load_yaml(jv_path)}"/> <!-- Read in the yaml dict as mp (short for model parameters) -->
+        <xacro:joint_configuration joint_name="${arm_id}_joint1" initial_position="${jv['panda_joint1']}"/>
+        <xacro:joint_configuration joint_name="${arm_id}_joint2" initial_position="${jv['panda_joint2']}"/>
+        <xacro:joint_configuration joint_name="${arm_id}_joint3" initial_position="${jv['panda_joint3']}"/>
+        <xacro:joint_configuration joint_name="${arm_id}_joint4" initial_position="${jv['panda_joint4']}"/>
+        <xacro:joint_configuration joint_name="${arm_id}_joint5" initial_position="${jv['panda_joint5']}"/>
+        <xacro:joint_configuration joint_name="${arm_id}_joint6" initial_position="${jv['panda_joint6']}"/>
+        <xacro:joint_configuration joint_name="${arm_id}_joint7" initial_position="${jv['panda_joint7']}"/>
         <!--
-        <xacro:configure_joint joint_name="${ns}_joint1" initial_position="0.0}"/>
-        <xacro:configure_joint joint_name="${ns}_joint2" initial_position="${-pi/4}"/>
-        <xacro:configure_joint joint_name="${ns}_joint3" initial_position="0.0"/>
-        <xacro:configure_joint joint_name="${ns}_joint4" initial_position="${-3*pi/4}"/>
-        <xacro:configure_joint joint_name="${ns}_joint5" initial_position="0.0"/>
-        <xacro:configure_joint joint_name="${ns}_joint6" initial_position="${pi/2}"/>
-        <xacro:configure_joint joint_name="${ns}_joint7" initial_position="${pi/4}"/>
         <joint name="panda_joint1">
             <command_interface name="effort">

File: franka_description/robots/panda_arm.ros2_control.xacro (robot description, xacro)
@@ -1,5 +1,5 @@
 <?xml version="1.0"?>
 <robot xmlns:xacro="http://www.ros.org/wiki/xacro">
-  <xacro:macro name="panda_arm_ros2_control" params="ns robot_ip use_fake_hardware:=^|false fake_sensor_commands:=^|false">
+  <xacro:macro name="panda_arm_ros2_control" params="ns robot_ip use_fake_hardware:=^|false fake_sensor_commands:=^|false ">
     <ros2_control name="FrankaHardwareInterface" type="system">
       <hardware>
@@ -16,14 +16,27 @@
       <xacro:macro name="configure_joint" params="joint_name initial_position">
         <joint name="${joint_name}">
-          <param name="initial_position">${initial_position}</param>
           <command_interface name="effort"/>
           <command_interface name="velocity"/>
           <command_interface name="position"/>
-          <state_interface name="position"/>
+          <state_interface name="position">
+            <param name="initial_position">${initial_position}</param>
+          </state_interface>
           <state_interface name="velocity"/>
           <state_interface name="effort"/>
         </joint>
       </xacro:macro>
-      <xacro:configure_joint joint_name="${ns}_joint1" initial_position="0.0"/>
+      <xacro:arg name="initial_joint_values_path" default=""/> <!-- Need argument to get from launch file -->
+      <xacro:property name="jv_path" value="$(arg initial_joint_values_path)"/> <!-- Need seperate property for xacro inorder processing -->
+      <xacro:property name="jv" value="${xacro.load_yaml(jv_path)}"/> <!-- Read in the yaml dict as mp (short for model parameters) -->
+      <!--
+      <xacro:configure_joint joint_name="${ns}_joint1" initial_position="${jv['panda_joint1']}"/>
+      <xacro:configure_joint joint_name="${ns}_joint2" initial_position="${jv['panda_joint2']}"/>
+      <xacro:configure_joint joint_name="${ns}_joint3" initial_position="${jv['panda_joint3']}"/>
+      <xacro:configure_joint joint_name="${ns}_joint4" initial_position="${jv['panda_joint4']}"/>
+      <xacro:configure_joint joint_name="${ns}_joint5" initial_position="${jv['panda_joint5']}"/>
+      <xacro:configure_joint joint_name="${ns}_joint6" initial_position="${jv['panda_joint6']}"/>
+      <xacro:configure_joint joint_name="${ns}_joint7" initial_position="${jv['panda_joint7']}"/>
+-->
+      <xacro:configure_joint joint_name="${ns}_joint1" initial_position="0.0}"/>
       <xacro:configure_joint joint_name="${ns}_joint2" initial_position="${-pi/4}"/>
       <xacro:configure_joint joint_name="${ns}_joint3" initial_position="0.0"/>

File: franka_description/robots/panda_arm.urdf.xacro (robot description, xacro)
@@ -4,6 +4,6 @@
   <xacro:arg name="hand" default="false"/> <!-- Should a franka_gripper be mounted at the flange?" -->
   <xacro:arg name="robot_ip" default=""/> <!-- IP address or hostname of the robot" -->
-  <xacro:arg name="use_fake_hardware" default="false"/>
-  <xacro:arg name="fake_sensor_commands" default="false"/>
+  <xacro:arg name="use_fake_hardware" default="true"/>
+  <xacro:arg name="fake_sensor_commands" default="true"/>
   <link name="world"/>
   <xacro:include filename="$(find franka_description)/robots/panda_arm.xacro"/>
@@ -15,5 +15,7 @@
   <xacro:include filename="$(find franka_description)/robots/manipulator.gazebo.xacro" />
   <xacro:include filename="$(find franka_description)/robots/manipulator.control.xacro" />
+  <!--
   <xacro:include filename="$(find franka_description)/robots/panda_arm.ros2_control.xacro"/>
   <xacro:panda_arm_ros2_control ns="$(arg arm_id)" robot_ip="$(arg robot_ip)" use_fake_hardware="$(arg use_fake_hardware)" fake_sensor_commands="$(arg fake_sensor_commands)"/>
+-->
 </robot>
